File: hardware/geulis.kicad_pcb (KiCad board)
At the start: 2 copper layers, 337.2 x 122.6 mm, 322 parts, among them J1 USB_C_Receptacle_USB2.0, J2 USB_C_Receptacle_USB2.0, J3 Conn_01x04, J4 Conn_01x02, J5 Conn_01x04, Q2 AO3407, Q3 AO3407, SW1 SW_PUSH, SW10 SW_PUSH, SW11 SW_PUSH, SW12 SW_PUSH, SW13 SW_PUSH, SW14 SW_PUSH, SW14_2 SW_PUSH, SW15 SW_PUSH, SW16 SW_PUSH, SW17 SW_PUSH, SW18 SW_PUSH, SW19 SW_PUSH, SW2 SW_PUSH, SW20 SW_PUSH, SW21 SW_PUSH, SW22 SW_PUSH, SW23 SW_PUSH, SW24 SW_PUSH, SW25 SW_PUSH, SW26 SW_PUSH, SW27 SW_PUSH, SW28 SW_PUSH, SW29 SW_PUSH, SW29_2 Rotary_Encoder_Switch, SW3 SW_PUSH, SW30 SW_PUSH, SW30_2 SW_PUSH, SW31 SW_PUSH, SW32 SW_PUSH, SW33 SW_PUSH, SW34 SW_PUSH, SW35 SW_PUSH, SW36 SW_PUSH, SW37 SW_PUSH, SW38 SW_PUSH, SW39 SW_PUSH, SW4 SW_PUSH, SW40 SW_PUSH, SW41 SW_PUSH, SW42 SW_PUSH, SW43 SW_PUSH, SW44 SW_PUSH, SW45 SW_PUSH, SW46 SW_PUSH, SW47 SW_PUSH, SW48 SW_PUSH, SW49 SW_PUSH, SW5 SW_PUSH, SW50 SW_PUSH, SW51 SW_PUSH, SW52 SW_PUSH, SW53 SW_PUSH, SW54 SW_PUSH, SW55 SW_PUSH, SW55_2 SW_PUSH, SW56 SW_PUSH, SW57 SW_PUSH, SW58 SW_PUSH, SW58_2 Rotary_Encoder_Switch, SW59 SW_PUSH, SW6 SW_PUSH, SW60 SW_PUSH, SW61 SW_PUSH, SW61_2 SW_PUSH, SW62 SW_PUSH, SW62_2 SW_PUSH, SW63 SW_PUSH, SW64 SW_PUSH, SW65 SW_PUSH, SW66 SW_PUSH, SW67 SW_SPDT, SW7 SW_PUSH, SW8 SW_PUSH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

Commit message: update
Parts:
- removed C22, C23, C24, C25, C26, C27, C28, C29, C30, C31, C32, C33, C34, C35, C36, C37, C38, C39, C40, C41, C42, C43, C44, C45, C46, C47, C48, C49, C50, C51, C52, C53, C54, C55, C56, C57, C58, C59, C60, C61, C62, C63, C64, C65, C66, C67, C68, C69, C70, C71, C72, C73, C74, C75, C76, C77, C78, C79, C80, C81, C82, C83, C84, C85, C86: 0.1uF, Capacitor_SMD:C_0805_2012Metric_Pad1.18x1.45mm_HandSolder
- removed D100, D101, D102, D103, D104, D105, D106, D107, D108, D109, D110, D111, D112, D113, D114, D115, D116, D117, D118, D119, D120, D121, D122, D123, D124, D125, D55, D56, D57, D58, D59, D60, D61, D62, D63, D64, D65, D66, D67, D68, D69, D70, D71, D72, D73, D74, D75, D76, D77, D78, D79, D80, D81, D82, D83, D84, D85, D86, D87, D88, D89, D90, D91, D92, D93, D94, D95, D96, D97, D98, D99: WS2812B, kbd:YS-SK6812MINI-E
- removed H9: MountingHole, MountingHole:MountingHole_2.2mm_M2_Pad
- removed SW_RESET2: SW_PUSH, Button_Switch_SMD:SW_SPST_TL3342
- removed U3: E73-2G4M08S1C-52840, nrfmicro:E73-2G4M08S1C-52840
- removed Y2: 32.768KHZ, Crystal:Crystal_SMD_3215-2Pin_3.2x1.5mm
- added BZ1: Buzzer, buzzer_12mm:PKLCS1212E2000-R1, B.Cu at (294.0, -42.1)
- added C87: 2.2uF, Capacitor_SMD:C_0805_2012Metric_Pad1.18x1.45mm_HandSolder, B.Cu at (204.7, -123.1)
- added D126: BLUE, LED_THT:LED_D3.0mm, F.Cu at (22.1, -38.8)
- added D127: GREEN, LED_THT:LED_D3.0mm, F.Cu at (22.1, -34.3)
- added D128: ORANGE, LED_THT:LED_D3.0mm, F.Cu at (22.1, -43.3)
- added D129: GREEN, LED_SMD:LED_0603_1608Metric_Pad1.05x0.95mm_HandSolder, F.Cu at (23.4, -34.3)
- added J6: Conn_01x05, Connector_PinHeader_2.54mm:PinHeader_1x05_P2.54mm_Vertical, B.Cu at (204.7, -119.1)
- added J7: Conn_01x04, Connector_PinHeader_2.00mm:PinHeader_1x04_P2.00mm_Vertical, F.Cu at (192.0, -38.9)
- added J8: Conn_01x03, Connector_PinHeader_2.00mm:PinHeader_1x03_P2.00mm_Vertical, F.Cu at (192.0, -32.7)
- added J9: Conn_01x04, Connector_PinHeader_2.00mm:PinHeader_1x04_P2.00mm_Vertical, F.Cu at (192.0, -35.8)
- added JP1: Jumper_2_Open, kbd:Jumper, B.Cu at (168.0, -124.3)
- added JP2: Jumper_2_Open, kbd:Jumper, B.Cu at (170.0, -124.3)
- added JP3: Jumper_2_Open, kbd:Jumper, B.Cu at (280.6, -42.5)
- added JP4: Jumper_2_Open, kbd:Jumper, B.Cu at (280.6, -39.6)
- added JP5: Jumper_2_Open, kbd:Jumper, B.Cu at (168.0, -126.7)
- added JP6: Jumper_2_Open, kbd:Jumper, B.Cu at (170.0, -126.7)
- added R1: 1K, Resistor_SMD:R_0603_1608Metric_Pad0.98x0.95mm_HandSolder, B.Cu at (23.3, -36.5)
- added R11: 100k, Resistor_SMD:R_0603_1608Metric_Pad0.98x0.95mm_HandSolder, B.Cu at (202.7, -122.9)
- added R12: 4.7k, Resistor_SMD:R_0603_1608Metric_Pad0.98x0.95mm_HandSolder, B.Cu at (196.8, -122.0)
- added R13: 4.7k, Resistor_SMD:R_0603_1608Metric_Pad0.98x0.95mm_HandSolder, B.Cu at (200.2, -122.0)
- added U1: nRF52840_holyiot_18010, kicad-keyboard-parts:nRF52840_holyiot_18010, B.Cu at (183.3, -67.5)
- D34, D35, D36, D37, D38, D39, D40, D41, D42, D43, D44, D45, D46, D47, D48, D49, D50, D51: footprint Keebio-Parts:WS2812B -> WS2812B:WS2812B_data-bridgeable
- D53, OL1: moved to F.Cu
- D54: value RED -> ORANGE; moved to F.Cu
- SW55_2: footprint MX_Alps_Hybrid-master:MXOnly-2.75U-Hotswap -> MX_Alps_Hybrid-master:MXOnly-2.75U-Hotswap-ReversedStabilizers
- moved H2 469.5 mm to (50.7, -110.7)
- moved C8 461.9 mm to (28.8, -64.5), turned to 180 degrees
- moved C12 445.6 mm to (77.5, -126.6), turned to 90 degrees
- moved H5 431.3 mm to (39.6, -51.1)
- moved H12 427.4 mm to (118.2, -105.9)
- moved H13 405.6 mm to (101.5, -50.3)
- moved D38 391.9 mm to (252.5, -126.5)
- moved H3 391.9 mm to (189.1, -100.4), turned to 204 degrees
- moved H10 361.1 mm to (346.8, -108.3)
- moved C5 358.6 mm to (164.5, -123.5), turned to 270 degrees
- moved H7 358.2 mm to (264.3, -106.7)
- moved C16 344.9 mm to (27.8, -120.0)
- moved D39 344.2 mm to (309.9, -126.4)
- moved H4 338.5 mm to (189.7, -24.9)
- moved C13 321.0 mm to (257.3, -126.5), turned to 270 degrees
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Connections:
- C1 pad 2: EXT_VCC -> UNDERGLOW_POWER
- C10 pad 1: EXT_VCC -> UNDERGLOW_POWER
- C11 pad 2: EXT_VCC -> UNDERGLOW_POWER
- C12 pad 2: EXT_VCC -> UNDERGLOW_POWER
- C13 pad 1: EXT_VCC -> UNDERGLOW_POWER
- C14 pad 1: EXT_VCC -> UNDERGLOW_POWER
- C15 pad 1: EXT_VCC -> UNDERGLOW_POWER
- C16 pad 2: EXT_VCC -> UNDERGLOW_POWER
- C17 pad 1: EXT_VCC -> UNDERGLOW_POWER
- C2 pad 2: EXT_VCC -> UNDERGLOW_POWER
- C21 pad 1: GND -> UNDERGLOW_POWER
- C21 pad 2: EXT_VCC -> GND
- C3 pad 1: EXT_VCC -> UNDERGLOW_POWER
- C4 pad 2: EXT_VCC -> UNDERGLOW_POWER
- C5 pad 1: EXT_VCC -> UNDERGLOW_POWER
- C6 pad 2: EXT_VCC -> UNDERGLOW_POWER
- C7 pad 1: EXT_VCC -> UNDERGLOW_POWER
- C8 pad 2: EXT_VCC -> UNDERGLOW_POWER
- C9 pad 1: EXT_VCC -> UNDERGLOW_POWER
- D34 pad 1: EXT_VCC -> UNDERGLOW_POWER
- D35 pad 1: EXT_VCC -> UNDERGLOW_POWER
- D36 pad 1: EXT_VCC -> UNDERGLOW_POWER
- D37 pad 1: EXT_VCC -> UNDERGLOW_POWER
- D38 pad 1: EXT_VCC -> UNDERGLOW_POWER
- D39 pad 1: EXT_VCC -> UNDERGLOW_POWER
- D40 pad 1: EXT_VCC -> UNDERGLOW_POWER
- D41 pad 1: EXT_VCC -> UNDERGLOW_POWER
- D42 pad 1: EXT_VCC -> UNDERGLOW_POWER
- D43 pad 1: EXT_VCC -> UNDERGLOW_POWER
- D44 pad 1: EXT_VCC -> UNDERGLOW_POWER
- D45 pad 1: EXT_VCC -> UNDERGLOW_POWER
- D46 pad 1: EXT_VCC -> UNDERGLOW_POWER
- D47 pad 1: EXT_VCC -> UNDERGLOW_POWER
- D48 pad 1: EXT_VCC -> UNDERGLOW_POWER
- D49 pad 1: EXT_VCC -> UNDERGLOW_POWER
- D50 pad 1: EXT_VCC -> UNDERGLOW_POWER
- D51 pad 1: EXT_VCC -> UNDERGLOW_POWER
- J3 pad 2: GND -> SWD
- J3 pad 3: SWD -> SWC
- J3 pad 4: SWC -> GND
- OL1 pad 3: EXT_VCC -> OLED_POWER
Routing:
- net EXT_VCC: track 1164.4 -> 205.7 mm, vias 3 -> 4
- net UNDERGLOW_POWER: track 0.00 -> 869.5 mm, vias 0 -> 10
- net r9: track 11.4 -> 477.1 mm, vias 0 -> 3
- net VBUS: track 0.00 -> 281.4 mm, vias 0 -> 4
- net GND: track 1376.1 -> 1115.3 mm, vias 3 -> 14
- net nRF_VDD: track 0.00 -> 248.4 mm, vias 0 -> 4
- net Net-(R9-Pad2): track 0.00 -> 223.1 mm, vias 0 -> 2
- net LED_INDICATOR2: track 0.00 -> 187.3 mm, vias 0 -> 1
- net LED_INDICATOR: track 0.00 -> 182.3 mm, vias 0 -> 1
- net r4: track 253.7 -> 431.7 mm, vias 0 -> 5
- net r8: track 375.3 -> 552.6 mm, vias 2 -> 5
- net rot1a: track 0.00 -> 169.6 mm, vias 0 -> 1
- net rot1b: track 0.00 -> 163.7 mm, vias 0 -> 1
- net rot3a: track 0.00 -> 158.0 mm, vias 0 -> 1
- net c6: track 110.0 -> 265.7 mm, vias 5 -> 4
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Other:
- outline, holes or cut-outs redrawn

Commit message: update
Parts:
- added G***: LOGO, geulis:geulis_text_negative, B.Cu at (84.5, -44.4)
- added G***: LOGO, geulis:geulis_text_negative, F.Cu at (84.9, -44.7)
- added JP7: vbat_switch, kbd:Jumper, F.Cu at (205.6, -34.3)
- JP1, JP3: value Jumper_2_Open -> nrf_vdd
- JP2, JP4: value Jumper_2_Open -> ext_vcc
- moved SW27 3.45 mm to (316.3, -98.4)
- moved D22 3.45 mm to (247.4, -93.9)
- moved J3 3.45 mm to (183.5, -123.0)
- moved J4 3.45 mm to (188.3, -52.6)
- moved J5 3.45 mm to (175.9, -125.4)
- moved JP6 3.45 mm to (173.5, -126.4)
- moved R13 3.45 mm to (203.7, -121.6)
- moved R3 3.45 mm to (187.9, -85.6)
- moved R6 3.45 mm to (188.1, -124.6)
- moved SW46 3.45 mm to (134.9, -54.8)
- moved SW6 3.45 mm to (160.8, -107.7)
- moved C10 3.45 mm to (81.5, -35.6)
- moved C12 3.45 mm to (81.0, -126.3)
- moved D1 3.45 mm to (73.2, -116.7)
- moved D8 3.45 mm to (98.4, -78.6)
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Connections:
- J7 pad 3: /P1.26 -> /P0.25
- J8 pad 1: /P0.16 -> /P0.13
- J8 pad 2: /P0.13 -> /P0.16
- J8 pad 3: /P0.14 -> /P0.19
- J9 pad 1: BUZZER_A -> /P1.14
- J9 pad 2: BUZZER_B -> /P1.07
- J9 pad 4: /P1.07 -> /P0.14
- U1 pad 20: Net-(U1-Pad20) -> /P0.19
- U1 pad 38: Net-(U1-Pad38) -> /P1.14
- U1 pad 40: Net-(U1-Pad40) -> /P0.25
Routing:
- net /P0.13: track 0.00 -> 76.7 mm, vias 0 -> 1
- net /P0.16: track 0.00 -> 71.7 mm, vias 0 -> 1
- net /P0.19: track 0.00 -> 60.8 mm, vias 0 -> 2
- net /P1.14: track 0.00 -> 59.1 mm, vias 0 -> 1
- net /P1.05: track 0.00 -> 51.9 mm
- net /P0.25: track 0.00 -> 50.9 mm, vias 0 -> 1
- net /P0.14: track 0.00 -> 49.7 mm, vias 0 -> 1
- net /P1.07: track 0.00 -> 49.3 mm
- net /P1.12: track 0.00 -> 45.7 mm, vias 0 -> 1
- net NFC1: track 0.00 -> 33.3 mm, vias 0 -> 1
- net NFC2: track 0.00 -> 31.9 mm, vias 0 -> 1
- net rot1s2: track 45.8 -> 54.9 mm
- net r1: track 350.6 -> 359.5 mm
- net r4: track 431.7 -> 439.4 mm
- net BUZZER_B: track 140.8 -> 146.4 mm
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- added copper zone on B.Cu, net GND
- added copper zone on F.Cu, net GND
Other:
- board text added: "013"
- board text added: "014"
- board text added: "016"
- board text added: "019"
- board text added: "025"
- board text added: "105"
- board text added: "107"
- board text added: "112"
- board text added: "114"
- board text added: "B+"
- board text added: "B-"
- board text added: "FREE PINS"
- board text added: "NFC1"
- board text added: "NFC2"

Commit message: add other file
Connections:
- net c0 renamed R0
- net c1 renamed R1
- net c2 renamed R2
- net c3 renamed R3
- net c4 renamed R4
- net c5 renamed R5
- net c6 renamed R6
- net r0 renamed C0
- net r1 renamed C1
- net r2 renamed C2
- net r3 renamed C3
- net r4 renamed C4
- net r5 renamed C5
- net r6 renamed C6
- net r7 renamed C7
- net r8 renamed C8
- net r9 renamed C9
Routing:
- net C0: track 343.5 -> 347.1 mm
- net (no net): track 0.00 -> 1.15 mm
- net R1: track 233.0 -> 233.5 mm
