File: hardware/geulis.sch (KiCad schematic (older format))
At the start: 322 parts, among them J1 USB_C_Receptacle_USB2.0, J2 USB_C_Receptacle_USB2.0, J3 Conn_01x04, J4 Conn_01x02, J5 Conn_01x04, Q2 AO3407, Q3 AO3407, SW1 SW_PUSH, SW10 SW_PUSH, SW11 SW_PUSH, SW12 SW_PUSH, SW13 SW_PUSH, SW14 SW_PUSH, SW14_2 SW_PUSH, SW15 SW_PUSH, SW16 SW_PUSH, SW17 SW_PUSH, SW18 SW_PUSH, SW19 SW_PUSH, SW2 SW_PUSH, SW20 SW_PUSH, SW21 SW_PUSH, SW22 SW_PUSH, SW23 SW_PUSH, SW24 SW_PUSH, SW25 SW_PUSH, SW26 SW_PUSH, SW27 SW_PUSH, SW28 SW_PUSH, SW29 SW_PUSH, SW29_2 Rotary_Encoder_Switch, SW3 SW_PUSH, SW30 SW_PUSH, SW30_2 SW_PUSH, SW31 SW_PUSH, SW32 SW_PUSH, SW33 SW_PUSH, SW34 SW_PUSH, SW35 SW_PUSH, SW36 SW_PUSH, SW37 SW_PUSH, SW38 SW_PUSH, SW39 SW_PUSH, SW4 SW_PUSH, SW40 SW_PUSH, SW41 SW_PUSH, SW42 SW_PUSH, SW43 SW_PUSH, SW44 SW_PUSH, SW45 SW_PUSH, SW46 SW_PUSH, SW47 SW_PUSH, SW48 SW_PUSH, SW49 SW_PUSH, SW5 SW_PUSH, SW50 SW_PUSH, SW51 SW_PUSH, SW52 SW_PUSH, SW53 SW_PUSH, SW54 SW_PUSH, SW55 SW_PUSH, SW55_2 SW_PUSH, SW56 SW_PUSH, SW57 SW_PUSH, SW58 SW_PUSH, SW58_2 Rotary_Encoder_Switch, SW59 SW_PUSH, SW6 SW_PUSH, SW60 SW_PUSH, SW61 SW_PUSH, SW61_2 SW_PUSH, SW62 SW_PUSH, SW62_2 SW_PUSH, SW63 SW_PUSH, SW64 SW_PUSH, SW65 SW_PUSH, SW66 SW_PUSH, SW67 SW_SPDT, SW7 SW_PUSH, SW8 SW_PUSH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

Commit message: update
Parts:
- removed C22, C23, C24, C25, C26, C27, C28, C29, C30, C31, C32, C33, C34, C35, C36, C37, C38, C39, C40, C41, C42, C43, C44, C45, C46, C47, C48, C49, C50, C51, C52, C53, C54, C55, C56, C57, C58, C59, C60, C61, C62, C63, C64, C65, C66, C67, C68, C69, C70, C71, C72, C73, C74, C75, C76, C77, C78, C79, C80, C81, C82, C83, C84, C85, C86: 0.1uF, Capacitor_SMD:C_0805_2012Metric_Pad1.18x1.45mm_HandSolder, symbol Device:C_Small
- removed D100, D101, D102, D103, D104, D105, D106, D107, D108, D109, D110, D111, D112, D113, D114, D115, D116, D117, D118, D119, D120, D121, D122, D123, D124, D125, D55, D56, D57, D58, D59, D60, D61, D62, D63, D64, D65, D66, D67, D68, D69, D70, D71, D72, D73, D74, D75, D76, D77, D78, D79, D80, D81, D82, D83, D84, D85, D86, D87, D88, D89, D90, D91, D92, D93, D94, D95, D96, D97, D98, D99: WS2812B, kbd:YS-SK6812MINI-E, symbol LED:WS2812B
- removed H9: MountingHole, MountingHole:MountingHole_2.2mm_M2_Pad, symbol Mechanical:MountingHole
- removed SW_RESET2: SW_PUSH, Button_Switch_SMD:SW_SPST_TL3342, symbol kbd:SW_PUSH
- removed U3: E73-2G4M08S1C-52840, nrfmicro:E73-2G4M08S1C-52840, symbol nrfmicro:E73-2G4M08S1C-52840
- removed Y2: 32.768KHZ, Crystal:Crystal_SMD_3215-2Pin_3.2x1.5mm, symbol Device:Crystal_Small
- added BZ1: Buzzer, buzzer_12mm:PKLCS1212E2000-R1, symbol Device:Buzzer
- added C87: 2.2uF, Capacitor_SMD:C_0805_2012Metric_Pad1.18x1.45mm_HandSolder, symbol Device:C_Small
- added D126: BLUE, LED_THT:LED_D3.0mm, symbol Device:LED
- added D127: GREEN, LED_THT:LED_D3.0mm, symbol Device:LED
- added D128: ORANGE, LED_THT:LED_D3.0mm, symbol Device:LED
- added D129: GREEN, LED_SMD:LED_0603_1608Metric_Pad1.05x0.95mm_HandSolder, symbol Device:LED
- added J6: Conn_01x05, Connector_PinHeader_2.54mm:PinHeader_1x05_P2.54mm_Vertical, symbol Connector_Generic:Conn_01x05
- added J7, J9: Conn_01x04, Connector_PinHeader_2.00mm:PinHeader_1x04_P2.00mm_Vertical, symbol Connector_Generic:Conn_01x04
- added J8: Conn_01x03, Connector_PinHeader_2.00mm:PinHeader_1x03_P2.00mm_Vertical, symbol Connector_Generic:Conn_01x03
- added JP1, JP2, JP3, JP4, JP5, JP6: Jumper_2_Open, kbd:Jumper, symbol Jumper:Jumper_2_Open
- added R1: 1K, Resistor_SMD:R_0603_1608Metric_Pad0.98x0.95mm_HandSolder, symbol Device:R_Small
- added R11: 100k, Resistor_SMD:R_0603_1608Metric_Pad0.98x0.95mm_HandSolder, symbol Device:R_Small
- added R12, R13: 4.7k, Resistor_SMD:R_0603_1608Metric_Pad0.98x0.95mm_HandSolder, symbol Device:R_Small
- added U1: nRF52840_holyiot_18010, kicad-keyboard-parts:nRF52840_holyiot_18010, symbol kicad-keyboard-parts:nRF52840_holyiot_18010
- D34, D35, D36, D37, D38, D39, D40, D41, D42, D43, D44, D45, D46, D47, D48, D49, D50, D51: footprint Keebio-Parts:WS2812B -> WS2812B:WS2812B_data-bridgeable
- D54: value RED -> ORANGE
- SW55_2: footprint MX_Alps_Hybrid-master:MXOnly-2.75U-Hotswap -> MX_Alps_Hybrid-master:MXOnly-2.75U-Hotswap-ReversedStabilizers
Connections:
- net BATTERY_PIN: now also U1.12 (P0.04)
- net DATA+: now also U1.24 (D+)
- net DATA-: now also U1.23 (D-)
- net EXT_VCC: now also JP2.2 (B), JP4.2 (B), JP6.2 (B); no longer C1.2, C10.1, C11.2, C12.2, C13.1, C14.1, C15.1, C16.2, C17.1, C2.2, C21.2, C3.1, C4.2, C5.1, C6.2, C7.1, C8.2, C9.1, D34.1 (VDD), D35.1 (VDD), D36.1 (VDD), D37.1 (VDD), D38.1 (VDD), D39.1 (VDD), D40.1 (VDD), D41.1 (VDD), D42.1 (VDD), D43.1 (VDD), D44.1 (VDD), D45.1 (VDD), D46.1 (VDD), D47.1 (VDD), D48.1 (VDD), D49.1 (VDD), D50.1 (VDD), D51.1 (VDD), OL1.3 (VCC)
- net GND: now also C21.2, J3.4 (Pin_4), J6.3 (Pin_3), R1.1, R11.2, U1.1 (GND), U1.25 (GND), U1.37 (GND); no longer C21.1, J3.2 (Pin_2)
- net LED_INDICATOR: now also D126.2 (A), U1.3 (P1.10)
- net LED_UNDERGLOW: now also U1.13 (P0.05)
- net P0.13: now also J8.2 (Pin_2), U1.54 (P0.13)
- net POWER_PIN: now also U1.16 (P1.09)
- net RESET: now also U1.21 (P0.18/RESET)
- net SCL: now also U1.51 (P0.17)
- net SDA: now also U1.52 (P0.15)
- net SWC: now also J3.3 (Pin_3), U1.31 (SWDCLK); no longer J3.4 (Pin_4)
- net SWD: now also J3.2 (Pin_2), U1.32 (SWDIO); no longer J3.3 (Pin_3)
- net VBUS: now also D128.2 (A), U1.22 (VBUS)
- net c0: now also U1.8 (P0.28)
- net c1: now also U1.5 (P1.15)
- net c2: now also U1.4 (P1.13)
- net c3: now also U1.33 (P1.04)
- net c4: now also U1.34 (P1.06)
- net c5: now also U1.30 (P1.02)
- net c6: now also U1.29 (P1.01)
- net nRF_VDD: now also JP1.2 (B), JP3.2 (B), JP5.2 (B), U1.14 (VDD_nRF)
- net r0: now also U1.19 (P0.21)
- net r1: now also U1.18 (P0.23)
- net r2: now also U1.15 (P0.07)
- net r3: now also U1.17 (P0.12)
- net r4: now also U1.7 (P0.02)
- net r5: now also U1.6 (P0.03)
- net r6: now also U1.28 (P1.03)
- net r7: now also U1.11 (P0.31)
- net r8: now also U1.9 (P0.29)
- net r9: now also U1.10 (P0.30)
- net rot1a: now also U1.45 (P0.06)
- net rot1b: now also U1.46 (P0.26)
- net rot2a: now also U1.44 (P0.08)
- net rot2b: now also U1.43 (P0.27)
- net rot3a: now also U1.42 (P1.08)
- net rot3b: now also U1.41 (P0.11)
- net at D53.1 (K), R8.2: now also D126.1 (K)
- net at D54.1 (K), R9.1: now also D128.1 (K)
- new net: D127.1 (K), D129.1 (K), R1.2
- new net BUZZER_A: BZ1.1 (-), J9.1 (Pin_1), U1.50 (P0.20)
- new net BUZZER_B: BZ1.2 (+), J9.2 (Pin_2), U1.49 (P0.24)
- new net LED_INDICATOR2: D127.2 (A), D129.2 (A), U1.2 (P1.11)
- new net NFC1: J7.2 (Pin_2), U1.35 (P0.09)
- new net NFC2: J7.1 (Pin_1), U1.36 (P0.10)
- new net OLED_POWER: JP3.1 (A), JP4.1 (A), OL1.3 (VCC)
- new net P0.14: J8.3 (Pin_3), U1.53 (P0.14)
- new net P0.16: J8.1 (Pin_1), U1.55 (P0.16)
- new net P1.05: J9.3 (Pin_3), U1.48 (P1.05)
- new net P1.07: J9.4 (Pin_4), U1.47 (P1.07)
- new net P1.12: J7.4 (Pin_4), U1.39 (P1.12)
- new net P1.26: J7.3 (Pin_3)
- new net TRACPOINT_POWER: C87.2, J6.4 (Pin_4), JP1.1 (A), JP2.1 (A), R12.1, R13.1
- new net T_CLK: J6.5 (Pin_5), R12.2, U1.26 (P0.22)
- new net T_DATA: J6.2 (Pin_2), R13.2, U1.27 (P1.00)
- new net UNDERGLOW_POWER: C1.2, C10.1, C11.2, C12.2, C13.1, C14.1, C15.1, C16.2, C17.1, C2.2, C21.1, C3.1, C4.2, C5.1, C6.2, C7.1, C8.2, C9.1, D34.1 (VDD), D35.1 (VDD), D36.1 (VDD), D37.1 (VDD), D38.1 (VDD), D39.1 (VDD), D40.1 (VDD), D41.1 (VDD), D42.1 (VDD), D43.1 (VDD), D44.1 (VDD), D45.1 (VDD), D46.1 (VDD), D47.1 (VDD), D48.1 (VDD), D49.1 (VDD), D50.1 (VDD), D51.1 (VDD), JP5.1 (A), JP6.1 (A)
- new net treset: C87.1, J6.1 (Pin_1), R11.1
- no-connect marks 3 -> 6
Other:
- moved on the sheet: D1, D10, D11, D12, D13, D14, D15, D16, D17, D18, D19, D2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

Commit message: update
Parts:
- added JP7: vbat_switch, kbd:Jumper, symbol Jumper:Jumper_2_Open
- JP1, JP3: value Jumper_2_Open -> nrf_vdd
- JP2, JP4: value Jumper_2_Open -> ext_vcc
Connections:
- net P1.26 is gone; now on net P0.25: J7.3 (Pin_3)
- net BUZZER_A: no longer J9.1 (Pin_1)
- net BUZZER_B: no longer J9.2 (Pin_2)
- net P0.13: now also J8.1 (Pin_1); no longer J8.2 (Pin_2)
- net P0.14: now also J9.4 (Pin_4); no longer J8.3 (Pin_3)
- net P0.16: now also J8.2 (Pin_2); no longer J8.1 (Pin_1)
- net P1.07: now also J9.2 (Pin_2); no longer J9.4 (Pin_4)
- net P1.14: now also J9.1 (Pin_1), U1.38 (P1.14)
- net VBAT: now also JP7.2 (B)
- net at Q2.3 (D), R3.1, SW67.3 (C): now also JP7.1 (A)
- net P0.19: now reaches U1.20 (P0.19)
- net P0.19: now also J8.3 (Pin_3)
- net P0.25: now reaches U1.40 (P0.25)
Other:
- moved on the sheet: BZ1, C87, D1, D10, D11, D12, D126, D127, D129, D13, D14, D15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

Commit message: add other file
Connections:
- net c0 renamed R0
- net c1 renamed R1
- net c2 renamed R2
- net c3 renamed R3
- net c4 renamed R4
- net c5 renamed R5
- net c6 renamed R6
- net r0 renamed C0
- net r1 renamed C1
- net r2 renamed C2
- net r3 renamed C3
- net r4 renamed C4
- net r5 renamed C5
- net r6 renamed C6
- net r7 renamed C7
- net r8 renamed C8
- net r9 renamed C9
